File: SegMan.kicad_pcb (KiCad board)
At the start: 2 copper layers, 50 parts, among them J1 Conn_01x02, J2 Conn_01x02, J3 Conn_01x02, J6 Conn_01x02, J7 Conn_01x02, K1 T9AS1D12-24, K2 T9AS1D12-24, Q1 BSS138W, Q2 BSS138W, U1 ADM6320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

Commit message: v1.0 of the PCB is done, oh, word?
Parts:
- removed D4: S1B, Diode_SMD:D_SMA_Handsoldering
- removed Q2: BSS138W, Package_TO_SOT_SMD:SOT-23_Handsoldering
- added C10: 0.1u, Capacitor_SMD:C_0805_2012Metric_Pad1.15x1.40mm_HandSolder, F.Cu at (190.2, 111.3)
- added G***: LOGO, Lafayette_Electric_Car_Footprints:segment, F.Cu at (185.2, 134.1)
- added G***: LOGO, Lafayette_Electric_Car_Footprints:highvoltagesmall, F.Cu at (82.8, 102.6)
- added G***: LOGO, Lafayette_Electric_Car_Footprints:highvoltage, B.Cu at (172.2, 75.9)
- added G***: LOGO, Lafayette_Electric_Car_Footprints:Paw, F.Cu at (185.2, 77.5)
- added G***: LOGO, Lafayette_Electric_Car_Footprints:ECE_Logo_Jon, F.Cu at (176.8, 69.6)
- added J3: CHRG-, Lafayette_Electric_Car_Footprints:DF22-1P-7.92, F.Cu at (94.6, 137.9)
- added J4: PacPower, Lafayette_Electric_Car_Footprints:DF22-2P-7.92, F.Cu at (99.1, 72.5)
- added REF**: MountingHole_4.5mm, MountingHole:MountingHole_4.5mm, F.Cu at (194.3, 141.7)
- added REF**: MountingHole_4.5mm, MountingHole:MountingHole_4.5mm, F.Cu at (82.5, 141.7)
- added REF**: MountingHole_4.5mm, MountingHole:MountingHole_4.5mm, F.Cu at (82.5, 68.1)
- added REF**: MountingHole_4.5mm, MountingHole:MountingHole_4.5mm, F.Cu at (194.3, 68.1)
- J1: value Conn_01x02 -> SegPower; footprint Lafayette_Electric_Car_Footprints:DF22R-2P-7.92 -> Lafayette_Electric_Car_Footprints:DF22-2P-7.92
- J2: value Conn_01x02 -> CHRG+; footprint Lafayette_Electric_Car_Footprints:DF22R-2P-7.92 -> Lafayette_Electric_Car_Footprints:DF22-1P-7.92
- J5: renamed from J3; value Conn_01x02 -> ChrgDetect
- J6: value Conn_01x02 -> I2CSeg; footprint Lafayette_Electric_Car_Footprints:DF22R-2P-7.92 -> Connector_PinHeader_2.54mm:PinHeader_1x04_P2.54mm_Vertical
- J7: value Conn_01x02 -> I2CPac; footprint Connector_PinHeader_2.54mm:PinHeader_1x02_P2.54mm_Vertical -> Connector_PinHeader_2.54mm:PinHeader_1x06_P2.54mm_Vertical
- R11: value 10k -> 22k
- moved C1 176.5 mm to (189.2, 101.1), turned to 270 degrees
- moved J7 169.9 mm to (193.0, 110.0)
- moved J5 169.4 mm to (193.0, 87.4)
- moved R7 117.8 mm to (153.4, 134.4), turned to 90 degrees
- moved TP6 117.5 mm to (184.9, 99.6), turned to 270 degrees
- moved TP4 116.4 mm to (185.7, 109.0)
- moved U1 105.3 mm to (161.8, 134.4)
- moved Q1 104.1 mm to (148.3, 134.4), turned to 180 degrees
- moved K1 101.6 mm to (135.3, 110.0)
- moved C3 100.5 mm to (157.5, 134.4), turned to 90 degrees
- moved J6 94.0 mm to (193.0, 97.3)
- moved D3 90.3 mm to (140.5, 134.4)
- moved F2 88.0 mm to (116.8, 68.1)
- moved F1 87.4 mm to (116.8, 73.8)
- moved R8 85.3 mm to (129.0, 70.7), turned to 180 degrees
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Connections:
- J6 pad 1: /VSEG+ -> /SEG_RTN
- J6 pad 2: /VSEG- -> /SCL_SEG
- J7 pad 1: /SEG_RTN -> /SEG_3V3
- J7 pad 2: /CHRG_DET -> /SDA_PAC
- K2 pad 2: Net-(D4-Pad2) -> Net-(D3-Pad2)
- R3 pad 2: /EN_CHRG -> /LED1
- R4 pad 2: /HEARTBEAT -> /LED2
- U4 pad 19: /HEARTBEAT -> Net-(U4-Pad19)
- U4 pad 28: /SCL_SEG -> /SDA_SEG
- U4 pad 29: /SDA_SEG -> /SCL_SEG
- U4 pad 4: Net-(U4-Pad4) -> /LED2
- U4 pad 5: Net-(U4-Pad5) -> /LED1
- U5 pad 1: /CurrentSensor+ -> /VSEG+
- U5 pad 2: /CurrentSensor+ -> /VSEG+
- U5 pad 3: /VSEG+ -> /CurrentSensor+
- U5 pad 4: /VSEG+ -> /CurrentSensor+
Routing:
- net /VSEG_FUSE_A: track 0.00 -> 252.7 mm
- net /SEG_5V: track 0.00 -> 116.3 mm, vias 0 -> 4
- net /SEG_3V3: track 0.00 -> 105.2 mm
- net /SEG_RTN: track 0.00 -> 82.2 mm, vias 0 -> 32
- net /~ALERT: track 0.00 -> 81.5 mm, vias 0 -> 1
- net /SDA_SEG: track 0.00 -> 80.2 mm
- net Net-(D3-Pad2): track 0.00 -> 78.7 mm, vias 0 -> 2
- net /SCL_SEG: track 0.00 -> 77.2 mm
- net /EN_CHRG: track 0.00 -> 58.7 mm, vias 0 -> 2
- net /VSEG-: track 0.00 -> 36.4 mm
- net /MISC_TO_PAC: track 0.00 -> 32.4 mm
- net /WATCHDOG: track 0.00 -> 31.8 mm
- net /VSEG_FUSE_B: track 0.00 -> 31.3 mm
- net /CURRENTSENSE: track 0.00 -> 31.3 mm
- net /VSEG+: track 0.00 -> 27.1 mm, vias 0 -> 16
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- added copper zone on B.Cu, net /CHRG+
- added copper zone on F.Cu, net /CHRG+
- added copper zone on B.Cu, net /CHRG-
- added copper zone on F.Cu, net /CHRG-
- added copper zone on B.Cu, net /CurrentSensor+
- added copper zone on F.Cu, net /CurrentSensor+
- added copper zone on B.Cu, net /SEG_RTN
- added copper zone on F.Cu, net /SEG_RTN
- added copper zone on B.Cu, net /VSEG+
- added copper zone on F.Cu, net /VSEG+
- added copper zone on B.Cu, net /VSEG-
- added copper zone on F.Cu, net /VSEG-
Other:
- board outline added: 121.9 x 83.8 mm
- rule trace_min: 0.25 -> 0.2
- board text added: "3.3V"
- board text added: "5.0V"
- board text added: "Charge Detect"
- board text added: "Charge+"
- board text added: "Charge-"
- board text added: "Jon Abel"
- board text added: "LED1"
- board text added: "LED2"
- board text added: "PacMan Power"
- board text added: "S/N"
- board text added: "SEG_RTN"
- board text added: "SegMan v1.0"
- board text added: "Segment Manager (SegMan) Fall 2019 Made in USA"
- board text added: "Segment Power"
- board text added: "To CellMen"
- board text added: "To PacMan"
- board text added: "VSEG+ A"
- board text added: "VSEG+ B"
- board text added: "Warning! Tractive System Voltage!"

Commit message: quick update before I retreat from the cave
Parts:
- moved R1 3.31 mm to (182.6, 100.3)
- moved R2 3.31 mm to (185.2, 100.3)
- moved TP6 3.31 mm to (185.2, 96.3)
- moved TP4 0.25 mm to (185.7, 109.2)
Routing:
- net /SCL_SEG: track 77.2 -> 80.3 mm
- net /SDA_SEG: track 80.2 -> 81.5 mm
- net /VSEG_FUSE_A: track 252.7 -> 253.2 mm
Other:
- board text added: "SCL"
- board text added: "SDA"
- board text added: "Unplug ESP8266 before plugging in USB!"

Commit message: the rise of ChordMan
Parts:
- removed D6: Q_SCR_AGK, Package_TO_SOT_SMD:SOT-23
- added D4: X0202MN 5BA4, Package_TO_SOT_SMD:SOT-223, F.Cu at (153.7, 74.4)
- D5: value D_Zener -> SMAZ5V6
- F1, F2: value 125mA -> 250mA; footprint Lafayette_Electric_Car_Footprints:0451.125MRL -> Lafayette_Electric_Car_Footprints:0154.500DRL
- moved D1 7.34 mm to (164.7, 82.9), turned to 180 degrees
- moved D2 6.88 mm to (164.7, 80.4), turned to 180 degrees
- moved TP5 6.56 mm to (160.3, 66.9)
- moved R3 2.91 mm to (160.7, 82.9), turned to 180 degrees
- moved G*** 1.52 mm to (173.7, 75.9)
- moved R4 1.41 mm to (160.7, 80.4), turned to 180 degrees
- moved F1 1.17 mm to (116.6, 74.9)
- moved F2 1.05 mm to (116.6, 69.1)
Routing:
- net /VSEG_FUSE_B: track 31.3 -> 43.5 mm
- net /SEG_RTN: track 82.2 -> 91.8 mm, vias 32 -> 30
- net /LED2: track 21.0 -> 23.1 mm
- net /LED1: track 24.6 -> 22.8 mm
- net /VSEG_FUSE_A: track 253.2 -> 252.7 mm
- net /VSEG+: track 27.1 -> 26.6 mm

Commit message: Lots of changes, no working version, somewhere in between 1.2 and 1.3
Parts:
- removed REF** (x4): MountingHole_4.5mm, MountingHole:MountingHole_4.5mm
- added H1: MountingHole_Pad, MountingHole:MountingHole_4.5mm_Pad, F.Cu at (152.2, 26.4)
- added H2: MountingHole_Pad, MountingHole:MountingHole_4.5mm_Pad, F.Cu at (152.2, 36.9)
- added H3: MountingHole_Pad, MountingHole:MountingHole_4.5mm_Pad, F.Cu at (162.8, 26.4)
- added H4: MountingHole_Pad, MountingHole:MountingHole_4.5mm_Pad, F.Cu at (167.0, 39.9)
- D1: value LED -> LED1
- D2: value LED -> LED2
Changed lines of the file:
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@@
   (general
     (thickness 1.6)
-    (drawings 30)
+    (drawings 28)
     (tracks 421)
     (zones 0)
     (modules 60)
-    (nets 42)
+    (nets 43)
   )
   (page A)
@@
   )
   (setup
-    (last_trace_width 0.5)
+    (last_trace_width 0.25)
     (user_trace_width 0.2)
     (user_trace_width 0.5)
@@
   (net 40 "Net-(J5-Pad2)")
   (net 41 "Net-(J5-Pad1)")
+  (net 42 /GLV_GND)
   (net_class Default "This is the default net class."
     (clearance 0.25)
@@
     (add_net /CurrentSensor+)
     (add_net /EN_CHRG)
+    (add_net /GLV_GND)
     (add_net /LED1)
     (add_net /LED2)
@@
       (xy -7.382718 2.7432) (xy -6.942559 2.7432) (xy -6.66062 2.759331)) (layer F.SilkS) (width 0.01))
   )
-  (module MountingHole:MountingHole_4.5mm (layer F.Cu)
-    (at 194.31 141.732)
-    (descr "Mounting Hole 4.5mm, no annular")
-    (tags "mounting hole 4.5mm no annular")
-    (attr virtual)
-    (fp_text reference REF** (at 0 -5.5) (layer F.SilkS) hide
-      (effects (font (size 1 1) (thickness 0.15)))
-    )
-    (fp_text value MountingHole_4.5mm (at 0 5.5) (layer F.Fab)
-      (effects (font (size 1 1) (thickness 0.15)))
-    )
-    (fp_circle (center 0 0) (end 4.75 0) (layer F.CrtYd) (width 0.05))
-    (fp_circle (center 0 0) (end 4.5 0) (layer Cmts.User) (width 0.15))
-    (fp_text user %R (at 0.3 0) (layer F.Fab)
-      (effects (font (size 1 1) (thickness 0.15)))
-    )
-    (pad 1 np_thru_hole circle (at 0 0) (size 4.5 4.5) (drill 4.5) (layers *.Cu *.Mask))
-  )
-  (module MountingHole:MountingHole_4.5mm (layer F.Cu)
-    (at 82.55 141.732)
-    (descr "Mounting Hole 4.5mm, no annular")
-    (tags "mounting hole 4.5mm no annular")
-    (attr virtual)
-    (fp_text reference REF** (at 0 -5.5) (layer F.SilkS) hide
-      (effects (font (size 1 1) (thickness 0.15)))
-    )
-    (fp_text value MountingHole_4.5mm (at 0 5.5) (layer F.Fab)
-      (effects (font (size 1 1) (thickness 0.15)))
-    )
-    (fp_circle (center 0 0) (end 4.75 0) (layer F.CrtYd) (width 0.05))
-    (fp_circle (center 0 0) (end 4.5 0) (layer Cmts.User) (width 0.15))
-    (fp_text user %R (at 0.3 0) (layer F.Fab)
-      (effects (font (size 1 1) (thickness 0.15)))
-    )
-    (pad 1 np_thru_hole circle (at 0 0) (size 4.5 4.5) (drill 4.5) (layers *.Cu *.Mask))
-  )
-  (module MountingHole:MountingHole_4.5mm (layer F.Cu)
-    (at 82.55 68.072)
-    (descr "Mounting Hole 4.5mm, no annular")
-    (tags "mounting hole 4.5mm no annular")
-    (attr virtual)
-    (fp_text reference REF** (at 0 -5.5) (layer F.SilkS) hide
-      (effects (font (size 1 1) (thickness 0.15)))
-    )
-    (fp_text value MountingHole_4.5mm (at 0 5.5) (layer F.Fab)
-      (effects (font (size 1 1) (thickness 0.15)))
-    )
-    (fp_circle (center 0 0) (end 4.75 0) (layer F.CrtYd) (width 0.05))
-    (fp_circle (center 0 0) (end 4.5 0) (layer Cmts.User) (width 0.15))
-    (fp_text user %R (at 0.3 0) (layer F.Fab)
-      (effects (font (size 1 1) (thickness 0.15)))
-    )
-    (pad 1 np_thru_hole circle (at 0 0) (size 4.5 4.5) (drill 4.5) (layers *.Cu *.Mask))
-  )
-  (module MountingHole:MountingHole_4.5mm (layer F.Cu)
-    (at 194.31 68.072)
-    (descr "Mounting Hole 4.5mm, no annular")
-    (tags "mounting hole 4.5mm no annular")
-    (attr virtual)
-    (fp_text reference REF** (at 0 6.858) (layer F.SilkS) hide
-      (effects (font (size 1 1) (thickness 0.15)))
-    )
-    (fp_text value MountingHole_4.5mm (at 0 5.5) (layer F.Fab)
-      (effects (font (size 1 1) (thickness 0.15)))
-    )
-    (fp_circle (center 0 0) (end 4.75 0) (layer F.CrtYd) (width 0.05))
-    (fp_circle (center 0 0) (end 4.5 0) (layer Cmts.User) (width 0.15))
-    (fp_text user %R (at 0.3 0) (layer F.Fab)
-      (effects (font (size 1 1) (thickness 0.15)))
-    )
-    (pad 1 np_thru_hole circle (at 0 0) (size 4.5 4.5) (drill 4.5) (layers *.Cu *.Mask))
-  )
   (module Lafayette_Electric_Car_Footprints:NodeMCUESP8266 (layer F.Cu)
     (at 154.305 92.583)
@@
       (effects (font (size 1 1) (thickness 0.15)))
     )
-    (fp_text value LED (at 0 1.43) (layer F.Fab)
+    (fp_text value LED2 (at 0 1.43) (layer F.Fab)
       (effects (font (size 1 1) (thickness 0.15)))
     )
@@
       (effects (font (size 1 1) (thickness 0.15)))
     )
-    (fp_text value LED (at 0 1.43) (layer F.Fab)
+    (fp_text value LED1 (at 0 1.43) (layer F.Fab)
       (effects (font (size 1 1) (thickness 0.15)))
     )
@@
     )
   )
+  (module MountingHole:MountingHole_4.5mm_Pad (layer F.Cu)
+    (at 152.222001 26.365001)
+    (descr "Mounting Hole 4.5mm")
+    (tags "mounting hole 4.5mm")
+    (attr virtual)
+    (fp_text reference H1 (at 0 -5.5) (layer F.SilkS)
+      (effects (font (size 1 1) (thickness 0.15)))
+    )
+    (fp_text value MountingHole_Pad (at 0 5.5) (layer F.Fab)
+      (effects (font (size 1 1) (thickness 0.15)))
+    )
+    (fp_circle (center 0 0) (end 4.75 0) (layer F.CrtYd) (width 0.05))
+    (fp_circle (center 0 0) (end 4.5 0) (layer Cmts.User) (width 0.15))
+    (fp_text user %R (at 0.3 0) (layer F.Fab)
+      (effects (font (size 1 1) (thickness 0.15)))
+    )
+    (pad 1 thru_hole circle (at 0 0) (size 9 9) (drill 4.5) (layers *.Cu *.Mask)
+      (net 42 /GLV_GND))
+  )
+  (module MountingHole:MountingHole_4.5mm_Pad (layer F.Cu)
+    (at 152.222001 36.915001)
+    (descr "Mounting Hole 4.5mm")
+    (tags "mounting hole 4.5mm")
+    (attr virtual)
+    (fp_text reference H2 (at 0 -5.5) (layer F.SilkS)
+      (effects (font (size 1 1) (thickness 0.15)))
+    )
+    (fp_text value MountingHole_Pad (at 0 5.5) (layer F.Fab)
+      (effects (font (size 1 1) (thickness 0.15)))
+    )
+    (fp_circle (center 0 0) (end 4.75 0) (layer F.CrtYd) (width 0.05))
+    (fp_circle (center 0 0) (end 4.5 0) (layer Cmts.User) (width 0.15))
+    (fp_text user %R (at 0.3 0) (layer F.Fab)
+      (effects (font (size 1 1) (thickness 0.15)))
+    )
+    (pad 1 thru_hole circle (at 0 0) (size 9 9) (drill 4.5) (layers *.Cu *.Mask)
+      (net 42 /GLV_GND))
+  )
+  (module MountingHole:MountingHole_4.5mm_Pad (layer F.Cu)
+    (at 162.772001 26.365001)
+    (descr "Mounting Hole 4.5mm")
+    (tags "mounting hole 4.5mm")
+    (attr virtual)
+    (fp_text reference H3 (at 0 -5.5) (layer F.SilkS)
+      (effects (font (size 1 1) (thickness 0.15)))
+    )
+    (fp_text value MountingHole_Pad (at 0 5.5) (layer F.Fab)
+      (effects (font (size 1 1) (thickness 0.15)))
+    )
+    (fp_text user %R (at 0.3 0) (layer F.Fab)
+      (effects (font (size 1 1) (thickness 0.15)))
+    )
+    (fp_circle (center 0 0) (end 4.5 0) (layer Cmts.User) (width 0.15))
+    (fp_circle (center 0 0) (end 4.75 0) (layer F.CrtYd) (width 0.05))
+    (pad 1 thru_hole circle (at 0 0) (size 9 9) (drill 4.5) (layers *.Cu *.Mask)
+      (net 42 /GLV_GND))
+  )
+  (module MountingHole:MountingHole_4.5mm_Pad (layer F.Cu)
+    (at 167.005 39.878)
+    (descr "Mounting Hole 4.5mm")
+    (tags "mounting hole 4.5mm")
+    (attr virtual)
+    (fp_text reference H4 (at 0 -5.5) (layer F.SilkS)
+      (effects (font (size 1 1) (thickness 0.15)))
+    )
+    (fp_text value MountingHole_Pad (at 0 5.5) (layer F.Fab)
+      (effects (font (size 1 1) (thickness 0.15)))
+    )
+    (fp_text user %R (at 0.3 0) (layer F.Fab)
+      (effects (font (size 1 1) (thickness 0.15)))
+    )
+    (fp_circle (center 0 0) (end 4.5 0) (layer Cmts.User) (width 0.15))
+    (fp_circle (center 0 0) (end 4.75 0) (layer F.CrtYd) (width 0.05))
+    (pad 1 thru_hole circle (at 0 0) (size 9 9) (drill 4.5) (layers *.Cu *.Mask)
+      (net 42 /GLV_GND))
+  )
   (gr_text "Jon Abel" (at 178.562 143.51) (layer F.Mask)
     (effects (font (size 2 2) (thickness 0.3) italic))
@@
     (effects (font (size 1 1) (thickness 0.15)))
   )
-  (dimension 83.82 (width 0.15) (layer Dwgs.User)
-    (gr_text "3.3 in" (at 205.77 104.902 270) (layer Dwgs.User)
-      (effects (font (size 1 1) (thickness 0.15)))
-    )
-    (feature1 (pts (xy 199.39 146.812) (xy 205.056421 146.812)))
-    (feature2 (pts (xy 199.39 62.992) (xy 205.056421 62.992)))
-    (crossbar (pts (xy 204.47 62.992) (xy 204.47 146.812)))
-    (arrow1a (pts (xy 204.47 146.812) (xy 203.883579 145.685496)))
-    (arrow1b (pts (xy 204.47 146.812) (xy 205.056421 145.685496)))
-    (arrow2a (pts (xy 204.47 62.992) (xy 203.883579 64.118504)))
-    (arrow2b (pts (xy 204.47 62.992) (xy 205.056421 64.118504)))
-  )
-  (dimension 121.92 (width 0.15) (layer Dwgs.User)
-    (gr_text "4.8 in" (at 138.43 56.612) (layer Dwgs.User)
-      (effects (font (size 1 1) (thickness 0.15)))
-    )
-    (feature1 (pts (xy 199.39 62.992) (xy 199.39 57.325579)))
-    (feature2 (pts (xy 77.47 62.992) (xy 77.47 57.325579)))
-    (crossbar (pts (xy 77.47 57.912) (xy 199.39 57.912)))
-    (arrow1a (pts (xy 199.39 57.912) (xy 198.263496 58.498421)))
-    (arrow1b (pts (xy 199.39 57.912) (xy 198.263496 57.325579)))
-    (arrow2a (pts (xy 77.47 57.912) (xy 78.596504 58.498421)))
-    (arrow2b (pts (xy 77.47 57.912) (xy 78.596504 57.325579)))
-  )
   (gr_line (start 77.47 146.812) (end 77.47 62.992) (layer Edge.Cuts) (width 0.05))
